Commit message: fix error

File: isuzu_vehicle_description/urdf/vehicle.xacro (robot description, xacro)
@@ -4,5 +4,5 @@
   <xacro:property
     name="vehicle_info"
-    value="${load_yaml('$(find isuzu_description)/config/vehicle_info.param.yaml')}"
+    value="${load_yaml('$(find isuzu_vehicle_description)/config/vehicle_info.param.yaml')}"
   />
   <!-- vehicle body -->
@@ -11,5 +11,5 @@
       <origin xyz="${vehicle_info['/**']['ros__parameters']['wheel_base']/2.0} 0 0" rpy="${pi/2.0} 0 ${pi/2.0}"/>
       <geometry>
-        <mesh filename="package://isuzu_description/mesh/isuzu.fbx" scale="0.01 0.01 0.01"/>
+        <mesh filename="package://isuzu_vehicle_description/mesh/isuzu.fbx" scale="0.01 0.01 0.01"/>
       </geometry>
     </visual>

Commit message: update vehicle model params

File: isuzu_vehicle_description/urdf/vehicle.xacro (robot description, xacro)
@@ -9,5 +9,6 @@
   <link name="base_link">
     <visual>
-      <origin xyz="${vehicle_info['/**']['ros__parameters']['wheel_base']/2.0} 0 0" rpy="${pi/2.0} 0 ${pi/2.0}"/>
+      <!--<origin xyz="${vehicle_info['/**']['ros__parameters']['wheel_base']/2.0} 0 0" rpy="${pi/2.0} 0 ${pi/2.0}"/>-->
+      <origin xyz="2.0772 0 -0.3935" rpy="${pi/2.0} 0 ${pi/2.0}"/>
       <geometry>
         <mesh filename="package://isuzu_vehicle_description/mesh/isuzu.fbx" scale="0.01 0.01 0.01"/>

Commit message: shift base_link on x axis

File: isuzu_vehicle_description/urdf/vehicle.xacro (robot description, xacro)
@@ -10,5 +10,5 @@
     <visual>
       <!--<origin xyz="${vehicle_info['/**']['ros__parameters']['wheel_base']/2.0} 0 0" rpy="${pi/2.0} 0 ${pi/2.0}"/>-->
-      <origin xyz="2.0772 0 -0.3935" rpy="${pi/2.0} 0 ${pi/2.0}"/>
+      <origin xyz="2.4772 0 -0.3935" rpy="${pi/2.0} 0 ${pi/2.0}"/>
       <geometry>
         <mesh filename="package://isuzu_vehicle_description/mesh/isuzu.fbx" scale="0.01 0.01 0.01"/>
